Commit message: Decimate Dorna TA meshes, fix URDF visual origins, rewrite README
- Re-decimate all Dorna TA STL meshes from original CAD exports
  (~5M faces -> 50-73k faces per link, 480 MB -> 19 MB total).
  Meshes remain in the CAD global frame.

- Fix mesh visualization: compute per-link visual origins that
  transform from CAD frame to each URDF link-local frame.
  Mapping: RotZ(-90deg) + cumulative FK translation.
  Previously meshes rendered as scattered parts due to incorrect
  identity rotation assumption.

- Add conditional visual elements in dorna_ta.urdf.xacro:
  mesh mode uses CAD-frame STLs with computed origins,
  primitive mode uses simple cylinders with identity origins.

- Rewrite README with accurate package layout, Docker/Foxglove
  setup, DH parameter table, mesh pipeline documentation, and
  architecture data flow diagram.

- Update display.launch.py for headless Docker operation
  (gui:=false runs joint_state_publisher without GUI/RViz).

- Add *.stl.orig to .gitignore (pre-decimation originals).

File: dorna2_description/urdf/dorna_ta.urdf.xacro (robot description, xacro)
@@ -28,26 +28,25 @@
     </inertial>
   </xacro:macro>
-  <!-- Visual/collision macro -->
-  <xacro:macro name="link_geometry" params="mesh_file fallback_length fallback_radius">
-    <xacro:if value="${use_mesh}">
-      <geometry>
-        <mesh filename="${mesh_file}" scale="0.001 0.001 0.001"/>
-      </geometry>
-    </xacro:if>
-    <xacro:unless value="${use_mesh}">
-      <geometry>
-        <cylinder length="${fallback_length}" radius="${fallback_radius}"/>
-      </geometry>
-    </xacro:unless>
-  </xacro:macro>
+  <!-- Mesh visual origin: transforms CAD-frame STLs into each link's local frame.
+       CAD frame to URDF mapping: RotZ(-90deg) + Z offset of d0. -->
+  <xacro:property name="mesh_yaw" value="${-PI/2}"/>
   <!-- World link (if standalone) -->
   <link name="$(arg parent)"/>
   <!-- Base link -->
   <link name="base_link">
-    <visual>
-      <origin xyz="0 0 0" rpy="0 0 0"/>
-      <xacro:link_geometry mesh_file="${mesh_dir}/base.stl" fallback_length="0.23" fallback_radius="0.06"/>
-      <material name="dorna_black"/>
-    </visual>
+    <xacro:if value="${use_mesh}">
+      <visual>
+        <origin xyz="0 0 ${d0}" rpy="0 0 ${mesh_yaw}"/>
+        <geometry><mesh filename="${mesh_dir}/base.stl" scale="0.001 0.001 0.001"/></geometry>
+        <material name="dorna_black"/>
+      </visual>
+    </xacro:if>
+    <xacro:unless value="${use_mesh}">
+      <visual>
+        <origin xyz="0 0 0" rpy="0 0 0"/>
+        <geometry><cylinder length="${d0}" radius="0.06"/></geometry>
+        <material name="dorna_black"/>
+      </visual>
+    </xacro:unless>
     <collision>
       <origin xyz="0 0 ${d0/2}" rpy="0 0 0"/>
@@ -65,9 +64,18 @@
   <!-- Joint 0: base rotation -->
   <link name="link0">
-    <visual>
-      <origin xyz="0 0 0" rpy="0 0 0"/>
-      <xacro:link_geometry mesh_file="${mesh_dir}/link0.stl" fallback_length="0.08" fallback_radius="0.04"/>
-      <material name="dorna_dark_grey"/>
-    </visual>
+    <xacro:if value="${use_mesh}">
+      <visual>
+        <origin xyz="0 0 0" rpy="0 0 ${mesh_yaw}"/>
+        <geometry><mesh filename="${mesh_dir}/link0.stl" scale="0.001 0.001 0.001"/></geometry>
+        <material name="dorna_dark_grey"/>
+      </visual>
+    </xacro:if>
+    <xacro:unless value="${use_mesh}">
+      <visual>
+        <origin xyz="0 0 0" rpy="0 0 0"/>
+        <geometry><cylinder length="0.08" radius="0.04"/></geometry>
+        <material name="dorna_dark_grey"/>
+      </visual>
+    </xacro:unless>
     <collision>
       <origin xyz="${a1/2} 0 0" rpy="0 ${PI/2} 0"/>
@@ -87,9 +95,18 @@
   <!-- Joint 1 -->
   <link name="link1">
-    <visual>
-      <origin xyz="0 0 0" rpy="0 0 0"/>
-      <xacro:link_geometry mesh_file="${mesh_dir}/link1.stl" fallback_length="0.21" fallback_radius="0.03"/>
-      <material name="dorna_dark_grey"/>
-    </visual>
+    <xacro:if value="${use_mesh}">
+      <visual>
+        <origin xyz="${-a1} 0 0" rpy="0 ${-PI/2} ${-PI/2}"/>
+        <geometry><mesh filename="${mesh_dir}/link1.stl" scale="0.001 0.001 0.001"/></geometry>
+        <material name="dorna_dark_grey"/>
+      </visual>
+    </xacro:if>
+    <xacro:unless value="${use_mesh}">
+      <visual>
+        <origin xyz="0 0 0" rpy="0 0 0"/>
+        <geometry><cylinder length="0.21" radius="0.03"/></geometry>
+        <material name="dorna_dark_grey"/>
+      </visual>
+    </xacro:unless>
     <collision>
       <origin xyz="${a2/2} 0 0" rpy="0 ${PI/2} 0"/>
@@ -109,9 +126,18 @@
   <!-- Joint 2 -->
   <link name="link2">
-    <visual>
-      <origin xyz="0 0 0" rpy="0 0 0"/>
-      <xacro:link_geometry mesh_file="${mesh_dir}/link2.stl" fallback_length="0.04" fallback_radius="0.03"/>
-      <material name="dorna_dark_grey"/>
-    </visual>
+    <xacro:if value="${use_mesh}">
+      <visual>
+        <origin xyz="${-(a1+a2)} 0 0" rpy="0 ${-PI/2} ${-PI/2}"/>
+        <geometry><mesh filename="${mesh_dir}/link2.stl" scale="0.001 0.001 0.001"/></geometry>
+        <material name="dorna_dark_grey"/>
+      </visual>
+    </xacro:if>
+    <xacro:unless value="${use_mesh}">
+      <visual>
+        <origin xyz="0 0 0" rpy="0 0 0"/>
+        <geometry><cylinder length="0.04" radius="0.03"/></geometry>
+        <material name="dorna_dark_grey"/>
+      </visual>
+    </xacro:unless>
     <collision>
       <origin xyz="0 0 ${d3/2}" rpy="0 0 0"/>
@@ -131,9 +157,18 @@
   <!-- Joint 3 -->
   <link name="link3">
-    <visual>
-      <origin xyz="0 0 0" rpy="0 0 0"/>
-      <xacro:link_geometry mesh_file="${mesh_dir}/link3.stl" fallback_length="0.175" fallback_radius="0.025"/>
-      <material name="dorna_dark_grey"/>
-    </visual>
+    <xacro:if value="${use_mesh}">
+      <visual>
+        <origin xyz="0 ${-d3} ${-(a1+a2)}" rpy="${PI/2} 0 ${PI/2}"/>
+        <geometry><mesh filename="${mesh_dir}/link3.stl" scale="0.001 0.001 0.001"/></geometry>
+        <material name="dorna_dark_grey"/>
+      </visual>
+    </xacro:if>
+    <xacro:unless value="${use_mesh}">
+      <visual>
+        <origin xyz="0 0 0" rpy="0 0 0"/>
+        <geometry><cylinder length="0.175" radius="0.025"/></geometry>
+        <material name="dorna_dark_grey"/>
+      </visual>
+    </xacro:unless>
     <collision>
       <origin xyz="0 0 ${d4/2}" rpy="0 0 0"/>
@@ -153,9 +188,18 @@
   <!-- Joint 4 -->
   <link name="link4">
-    <visual>
-      <origin xyz="0 0 0" rpy="0 0 0"/>
-      <xacro:link_geometry mesh_file="${mesh_dir}/link4.stl" fallback_length="0.089" fallback_radius="0.02"/>
-      <material name="dorna_dark_grey"/>
-    </visual>
+    <xacro:if value="${use_mesh}">
+      <visual>
+        <origin xyz="0 ${-(a1+a2+d4)} ${-d3}" rpy="0 ${-PI/2} 0"/>
+        <geometry><mesh filename="${mesh_dir}/link4.stl" scale="0.001 0.001 0.001"/></geometry>
+        <material name="dorna_dark_grey"/>
+      </visual>
+    </xacro:if>
+    <xacro:unless value="${use_mesh}">
+      <visual>
+        <origin xyz="0 0 0" rpy="0 0 0"/>
+        <geometry><cylinder length="0.089" radius="0.02"/></geometry>
+        <material name="dorna_dark_grey"/>
+      </visual>
+    </xacro:unless>
     <collision>
       <origin xyz="0 0 ${d5/2}" rpy="0 0 0"/>
@@ -175,9 +219,18 @@
   <!-- Joint 5 -->
   <link name="link5">
-    <visual>
-      <origin xyz="0 0 0" rpy="0 0 0"/>
-      <xacro:link_geometry mesh_file="${mesh_dir}/link5.stl" fallback_length="0.035" fallback_radius="0.018"/>
-      <material name="dorna_light_grey"/>
-    </visual>
+    <xacro:if value="${use_mesh}">
+      <visual>
+        <origin xyz="0 ${-d3-d5} ${-(a1+a2+d4)}" rpy="${PI/2} 0 ${PI/2}"/>
+        <geometry><mesh filename="${mesh_dir}/link5.stl" scale="0.001 0.001 0.001"/></geometry>
+        <material name="dorna_light_grey"/>
+      </visual>
+    </xacro:if>
+    <xacro:unless value="${use_mesh}">
+      <visual>
+        <origin xyz="0 0 0" rpy="0 0 0"/>
+        <geometry><cylinder length="0.035" radius="0.018"/></geometry>
+        <material name="dorna_light_grey"/>
+      </visual>
+    </xacro:unless>
     <collision>
       <origin xyz="0 0 ${d6/2}" rpy="0 0 0"/>

Commit message: Fixed TA

File: dorna2_description/urdf/dorna_ta.urdf.xacro (robot description, xacro)
@@ -28,7 +28,7 @@
     </inertial>
   </xacro:macro>
-  <!-- Mesh visual origin: transforms CAD-frame STLs into each link's local frame.
-       CAD frame to URDF mapping: RotZ(-90deg) + Z offset of d0. -->
-  <xacro:property name="mesh_yaw" value="${-PI/2}"/>
+  <!-- Visual origins: transform CAD-frame meshes into each link's local frame.
+       CAD frame -> URDF: RotZ(-PI/2) + Z offset of d0.
+       Per-link origin: T_link_inv @ T_cad at zero config. -->
   <!-- World link (if standalone) -->
   <link name="$(arg parent)"/>
@@ -37,5 +37,5 @@
     <xacro:if value="${use_mesh}">
       <visual>
-        <origin xyz="0 0 ${d0}" rpy="0 0 ${mesh_yaw}"/>
+        <origin xyz="0 0 ${d0}" rpy="0 0 ${-PI/2}"/>
         <geometry><mesh filename="${mesh_dir}/base.stl" scale="0.001 0.001 0.001"/></geometry>
         <material name="dorna_black"/>
@@ -66,5 +66,5 @@
     <xacro:if value="${use_mesh}">
       <visual>
-        <origin xyz="0 0 0" rpy="0 0 ${mesh_yaw}"/>
+        <origin xyz="0 0 0" rpy="0 0 ${-PI/2}"/>
         <geometry><mesh filename="${mesh_dir}/link0.stl" scale="0.001 0.001 0.001"/></geometry>
         <material name="dorna_dark_grey"/>
@@ -97,5 +97,5 @@
     <xacro:if value="${use_mesh}">
       <visual>
-        <origin xyz="${-a1} 0 0" rpy="0 ${-PI/2} ${-PI/2}"/>
+        <origin xyz="${-a1} 0 0" rpy="${-PI/2} ${-PI/2} 0"/>
         <geometry><mesh filename="${mesh_dir}/link1.stl" scale="0.001 0.001 0.001"/></geometry>
         <material name="dorna_dark_grey"/>
@@ -128,5 +128,5 @@
     <xacro:if value="${use_mesh}">
       <visual>
-        <origin xyz="${-(a1+a2)} 0 0" rpy="0 ${-PI/2} ${-PI/2}"/>
+        <origin xyz="${-(a1+a2)} 0 0" rpy="${-PI/2} ${-PI/2} 0"/>
         <geometry><mesh filename="${mesh_dir}/link2.stl" scale="0.001 0.001 0.001"/></geometry>
         <material name="dorna_dark_grey"/>
@@ -221,5 +221,5 @@
     <xacro:if value="${use_mesh}">
       <visual>
-        <origin xyz="0 ${-d3-d5} ${-(a1+a2+d4)}" rpy="${PI/2} 0 ${PI/2}"/>
+        <origin xyz="0 ${d5-d3} ${-(a1+a2+d4)}" rpy="${PI/2} 0 ${PI/2}"/>
         <geometry><mesh filename="${mesh_dir}/link5.stl" scale="0.001 0.001 0.001"/></geometry>
         <material name="dorna_light_grey"/>
