Commit message: Fix Dorna 2 visualization: merge arm meshes, compute visual origins
- Compute correct CAD-to-URDF visual origins for dorna_2.urdf.xacro
  based on Dorna_2.step global frame alignment (RotZ(+PI/2) + translation)
- Merge link1-link4 CAD assemblies into single link1.stl (100k faces)
  to prevent visual disconnection at articulated poses
- Replace link2-link4 with placeholder meshes (same approach as Dorna TA)
- Update README to reflect consolidated mesh strategy for both models

File: dorna2_description/urdf/dorna_2.urdf.xacro (robot description, xacro)
@@ -6,4 +6,12 @@
     Joint limits from Dorna 2 series user manual.
     model arg selects between "dorna_2" (d1=206.4mm) and "dorna_2s" (d1=218.47mm).
+    Mesh coordinate mapping: STLs are in the CAD global frame (Dorna_2.step).
+    CAD frame: arm extends in -Y, Z vertical, base axis at ~(19mm, 44.2mm) in XY.
+    Visual origins transform CAD geometry into each link's local frame via:
+      T_visual = T_world_link^{-1} @ T_cad_to_world
+    where T_cad_to_world = Trans(cad_tx, cad_ty, d1 - cad_arm_z) @ RotZ(+PI/2).
+    Link1 contains merged geometry from the original link1-link4 CAD assemblies.
+    Links 2-4 use placeholder meshes. Only joint0 (base rotation) and joint1
+    (shoulder pitch) produce visible mesh articulation.
   -->
   <xacro:include filename="$(find dorna2_description)/urdf/materials.xacro"/>
@@ -23,4 +31,9 @@
   <xacro:property name="a4" value="0.1524"/>
   <xacro:property name="d5" value="0.04892"/>
+  <!-- CAD frame alignment offsets (meters, after mesh 0.001 scale).
+       Derived from the base rotation axis position in the CAD export. -->
+  <xacro:property name="cad_tx" value="0.0442"/>
+  <xacro:property name="cad_ty" value="-0.019"/>
+  <xacro:property name="cad_arm_z" value="0.2423"/>
   <xacro:macro name="default_inertia" params="mass">
     <inertial>
@@ -29,24 +42,21 @@
     </inertial>
   </xacro:macro>
-  <xacro:macro name="link_geometry" params="mesh_file fallback_length fallback_radius">
-    <xacro:if value="${use_mesh}">
-      <geometry>
-        <mesh filename="${mesh_file}" scale="0.001 0.001 0.001"/>
-      </geometry>
-    </xacro:if>
-    <xacro:unless value="${use_mesh}">
-      <geometry>
-        <cylinder length="${fallback_length}" radius="${fallback_radius}"/>
-      </geometry>
-    </xacro:unless>
-  </xacro:macro>
   <link name="$(arg parent)"/>
   <!-- Base link -->
   <link name="base_link">
-    <visual>
-      <origin xyz="0 0 0" rpy="0 0 0"/>
-      <xacro:link_geometry mesh_file="${mesh_dir}/base.stl" fallback_length="${d1}" fallback_radius="0.05"/>
-      <material name="dorna_black"/>
-    </visual>
+    <xacro:if value="${use_mesh}">
+      <visual>
+        <origin xyz="${cad_tx} ${cad_ty} ${d1 - cad_arm_z}" rpy="0 0 ${PI/2}"/>
+        <geometry><mesh filename="${mesh_dir}/base.stl" scale="0.001 0.001 0.001"/></geometry>
+        <material name="dorna_black"/>
+      </visual>
+    </xacro:if>
+    <xacro:unless value="${use_mesh}">
+      <visual>
+        <origin xyz="0 0 0" rpy="0 0 0"/>
+        <geometry><cylinder length="${d1}" radius="0.05"/></geometry>
+        <material name="dorna_black"/>
+      </visual>
+    </xacro:unless>
     <collision>
       <origin xyz="0 0 ${d1/2}" rpy="0 0 0"/>
@@ -64,9 +74,18 @@
   <!-- Joint 0: base rotation -->
   <link name="link0">
-    <visual>
-      <origin xyz="0 0 0" rpy="0 0 0"/>
-      <xacro:link_geometry mesh_file="${mesh_dir}/link0.stl" fallback_length="0.095" fallback_radius="0.04"/>
-      <material name="dorna_dark_grey"/>
-    </visual>
+    <xacro:if value="${use_mesh}">
+      <visual>
+        <origin xyz="${cad_tx} ${cad_ty} ${-cad_arm_z}" rpy="0 0 ${PI/2}"/>
+        <geometry><mesh filename="${mesh_dir}/link0.stl" scale="0.001 0.001 0.001"/></geometry>
+        <material name="dorna_dark_grey"/>
+      </visual>
+    </xacro:if>
+    <xacro:unless value="${use_mesh}">
+      <visual>
+        <origin xyz="0 0 0" rpy="0 0 0"/>
+        <geometry><cylinder length="0.095" radius="0.04"/></geometry>
+        <material name="dorna_dark_grey"/>
+      </visual>
+    </xacro:unless>
     <collision>
       <origin xyz="${a2/2} 0 0" rpy="0 ${PI/2} 0"/>
@@ -84,11 +103,20 @@
     <limit lower="${-160*PI/180}" upper="${180*PI/180}" velocity="${225*PI/180}" effort="50"/>
   </joint>
-  <!-- Joint 1 -->
+  <!-- Joint 1: shoulder pitch. link1 carries merged arm geometry (link1-link4 CAD assemblies). -->
   <link name="link1">
-    <visual>
-      <origin xyz="0 0 0" rpy="0 0 0"/>
-      <xacro:link_geometry mesh_file="${mesh_dir}/link1.stl" fallback_length="0.203" fallback_radius="0.025"/>
-      <material name="dorna_dark_grey"/>
-    </visual>
+    <xacro:if value="${use_mesh}">
+      <visual>
+        <origin xyz="${cad_tx - a2} ${-cad_arm_z} ${-cad_ty}" rpy="${-PI/2} ${PI/2} 0"/>
+        <geometry><mesh filename="${mesh_dir}/link1.stl" scale="0.001 0.001 0.001"/></geometry>
+        <material name="dorna_dark_grey"/>
+      </visual>
+    </xacro:if>
+    <xacro:unless value="${use_mesh}">
+      <visual>
+        <origin xyz="0 0 0" rpy="0 0 0"/>
+        <geometry><cylinder length="0.203" radius="0.025"/></geometry>
+        <material name="dorna_dark_grey"/>
+      </visual>
+    </xacro:unless>
     <collision>
       <origin xyz="${a3/2} 0 0" rpy="0 ${PI/2} 0"/>
@@ -106,11 +134,20 @@
     <limit lower="${(-91 if model == 'dorna_2s' else -90)*PI/180}" upper="${(181 if model == 'dorna_2s' else 180)*PI/180}" velocity="${225*PI/180}" effort="50"/>
   </joint>
-  <!-- Joint 2 -->
+  <!-- Joint 2: placeholder mesh (geometry merged into link1) -->
   <link name="link2">
-    <visual>
-      <origin xyz="0 0 0" rpy="0 0 0"/>
-      <xacro:link_geometry mesh_file="${mesh_dir}/link2.stl" fallback_length="0.152" fallback_radius="0.02"/>
-      <material name="dorna_dark_grey"/>
-    </visual>
+    <xacro:if value="${use_mesh}">
+      <visual>
+        <origin xyz="0 0 0" rpy="0 0 0"/>
+        <geometry><mesh filename="${mesh_dir}/link2.stl" scale="0.001 0.001 0.001"/></geometry>
+        <material name="dorna_dark_grey"/>
+      </visual>
+    </xacro:if>
+    <xacro:unless value="${use_mesh}">
+      <visual>
+        <origin xyz="0 0 0" rpy="0 0 0"/>
+        <geometry><cylinder length="0.152" radius="0.02"/></geometry>
+        <material name="dorna_dark_grey"/>
+      </visual>
+    </xacro:unless>
     <collision>
       <origin xyz="${a4/2} 0 0" rpy="0 ${PI/2} 0"/>
@@ -128,11 +165,20 @@
     <limit lower="${-142*PI/180}" upper="${142*PI/180}" velocity="${240*PI/180}" effort="30"/>
   </joint>
-  <!-- Joint 3: wrist pitch -->
+  <!-- Joint 3: placeholder mesh -->
   <link name="link3">
-    <visual>
-      <origin xyz="0 0 0" rpy="0 0 0"/>
-      <xacro:link_geometry mesh_file="${mesh_dir}/link3.stl" fallback_length="0.049" fallback_radius="0.015"/>
-      <material name="dorna_dark_grey"/>
-    </visual>
+    <xacro:if value="${use_mesh}">
+      <visual>
+        <origin xyz="0 0 0" rpy="0 0 0"/>
+        <geometry><mesh filename="${mesh_dir}/link3.stl" scale="0.001 0.001 0.001"/></geometry>
+        <material name="dorna_dark_grey"/>
+      </visual>
+    </xacro:if>
+    <xacro:unless value="${use_mesh}">
+      <visual>
+        <origin xyz="0 0 0" rpy="0 0 0"/>
+        <geometry><cylinder length="0.049" radius="0.015"/></geometry>
+        <material name="dorna_dark_grey"/>
+      </visual>
+    </xacro:unless>
     <collision>
       <origin xyz="0 0 0" rpy="0 0 0"/>
@@ -150,11 +196,20 @@
     <limit lower="${-135*PI/180}" upper="${135*PI/180}" velocity="${1125*PI/180}" effort="10"/>
   </joint>
-  <!-- Joint 4: wrist roll (continuous) -->
+  <!-- Joint 4: wrist roll (continuous), placeholder mesh -->
   <link name="link4">
-    <visual>
-      <origin xyz="0 0 0" rpy="0 0 0"/>
-      <xacro:link_geometry mesh_file="${mesh_dir}/link4.stl" fallback_length="0.049" fallback_radius="0.012"/>
-      <material name="dorna_light_grey"/>
-    </visual>
+    <xacro:if value="${use_mesh}">
+      <visual>
+        <origin xyz="0 0 0" rpy="0 0 0"/>
+        <geometry><mesh filename="${mesh_dir}/link4.stl" scale="0.001 0.001 0.001"/></geometry>
+        <material name="dorna_light_grey"/>
+      </visual>
+    </xacro:if>
+    <xacro:unless value="${use_mesh}">
+      <visual>
+        <origin xyz="0 0 0" rpy="0 0 0"/>
+        <geometry><cylinder length="0.049" radius="0.012"/></geometry>
+        <material name="dorna_light_grey"/>
+      </visual>
+    </xacro:unless>
     <collision>
       <origin xyz="0 0 ${d5/2}" rpy="0 0 0"/>

Commit message: Better meshes

File: dorna2_description/urdf/dorna_2.urdf.xacro (robot description, xacro)
@@ -6,9 +6,6 @@
     Joint limits from Dorna 2 series user manual.
     model arg selects between "dorna_2" (d1=206.4mm) and "dorna_2s" (d1=218.47mm).
-    Mesh coordinate mapping: STLs are in the CAD global frame (Dorna_2.step).
-    CAD frame: arm extends in -Y, Z vertical, base axis at ~(19mm, 44.2mm) in XY.
-    Visual origins transform CAD geometry into each link's local frame via:
-      T_visual = T_world_link^{-1} @ T_cad_to_world
-    where T_cad_to_world = Trans(cad_tx, cad_ty, d1 - cad_arm_z) @ RotZ(+PI/2).
+    Meshes are pre-transformed from the CAD global frame (Dorna_2.step) into
+    each link's local URDF frame, so visual origins are identity.
     Link1 contains merged geometry from the original link1-link4 CAD assemblies.
     Links 2-4 use placeholder meshes. Only joint0 (base rotation) and joint1
@@ -31,9 +28,6 @@
   <xacro:property name="a4" value="0.1524"/>
   <xacro:property name="d5" value="0.04892"/>
-  <!-- CAD frame alignment offsets (meters, after mesh 0.001 scale).
-       Derived from the base rotation axis position in the CAD export. -->
-  <xacro:property name="cad_tx" value="0.0442"/>
-  <xacro:property name="cad_ty" value="-0.019"/>
-  <xacro:property name="cad_arm_z" value="0.2423"/>
+  <!-- Meshes are pre-transformed to each link's local frame.
+       No CAD-frame alignment needed; visual origins are identity. -->
   <xacro:macro name="default_inertia" params="mass">
     <inertial>
@@ -47,5 +41,5 @@
     <xacro:if value="${use_mesh}">
       <visual>
-        <origin xyz="${cad_tx} ${cad_ty} ${d1 - cad_arm_z}" rpy="0 0 ${PI/2}"/>
+        <origin xyz="0 0 0" rpy="0 0 0"/>
         <geometry><mesh filename="${mesh_dir}/base.stl" scale="0.001 0.001 0.001"/></geometry>
         <material name="dorna_black"/>
@@ -76,5 +70,5 @@
     <xacro:if value="${use_mesh}">
       <visual>
-        <origin xyz="${cad_tx} ${cad_ty} ${-cad_arm_z}" rpy="0 0 ${PI/2}"/>
+        <origin xyz="0 0 0" rpy="0 0 0"/>
         <geometry><mesh filename="${mesh_dir}/link0.stl" scale="0.001 0.001 0.001"/></geometry>
         <material name="dorna_dark_grey"/>
@@ -107,5 +101,5 @@
     <xacro:if value="${use_mesh}">
       <visual>
-        <origin xyz="${cad_tx - a2} ${-cad_arm_z} ${-cad_ty}" rpy="${-PI/2} ${PI/2} 0"/>
+        <origin xyz="0 0 0" rpy="0 0 0"/>
         <geometry><mesh filename="${mesh_dir}/link1.stl" scale="0.001 0.001 0.001"/></geometry>
         <material name="dorna_dark_grey"/>
